File: af-pj-bis2025.kicad_pcb (KiCad board)
At the start: 2 copper layers, 70 x 93.2 mm, 113 parts, among them J1 CN7, J10 Conn_01x02, J11 Conn_01x02, J2 CN10, J3 FH28-10S-0.5SH_05_, J4 Conn_02x05_Odd_Even, J5 Barrel_Jack_MountingPin, J6 Conn_Coaxial, J7 Conn_Coaxial, J8 Conn_01x02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

Commit message: DRCエラーフリー
Parts:
- moved R35 3.00 mm to (190.0, 137.0)
- moved R36 3.00 mm to (192.5, 137.0)
- moved R37 3.00 mm to (187.5, 137.0)
- moved C4 2.94 mm to (171.0, 81.5)
- moved C12 2.56 mm to (195.5, 73.0), turned to -90 degrees
Routing:
- net /DC_9V: track 47.8 -> 43.8 mm
- net GND: track 27.6 -> 23.9 mm, vias 96 -> 112
- net /ADC_MOSI: track 51.7 -> 54.7 mm
- net /ADC_MISO: track 52.5 -> 55.5 mm
- net /ADC_DRDY: track 44.1 -> 47.1 mm
- net /LCD_DISP: track 47.3 -> 49.7 mm, vias 4 -> 2
- net Net-(U8-*DRDY): track 8.65 -> 6.45 mm
- net /AVDD_5V: track 152.7 -> 150.8 mm
- net GNDA: track 70.2 -> 71.2 mm, vias 259 -> 265

Commit message: 基板完成
Parts:
- J4: footprint Connector_PinSocket_2.54mm:PinSocket_2x05_P2.54mm_Vertical -> Connector_PinHeader_2.54mm:PinHeader_2x05_P2.54mm_Vertical
- moved J4 2.58 mm to (158.6, 102.6)
Routing:
- net Net-(J4-Pin_9): track 20.3 -> 23.6 mm
- net Net-(J4-Pin_7): track 24.1 -> 26.6 mm
- net /LCD_DISP: track 49.7 -> 51.8 mm, vias 2 -> 5
- net +3V3: track 93.9 -> 95.8 mm
- net Net-(J4-Pin_8): track 24.8 -> 23.4 mm, vias 2 -> 4
- net Net-(J4-Pin_10): track 22.5 -> 21.4 mm
- net GNDA: vias 265 -> 292
- net GND: vias 112 -> 121
