File: stm32/stm32.kicad_sch (KiCad schematic)
At the start: 81 parts, among them J1 CN7, J2 CN10, J3 Conn_01x06, J4 Conn_Coaxial, J5 Barrel_Jack_MountingPin, J7 Conn_Coaxial, U1 MIC5237-5.0YU, U2 ALD114904APAL, U3 OPA2380AIDGKR, U4 THS4552IPWR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

Commit message: 差動増幅回路のレイアウト完了
Parts:
- removed J4, J7: Conn_Coaxial, Connector_Coaxial:SMA_Amphenol_901-143_Horizontal, symbol Connector:Conn_Coaxial
- removed J5: Barrel_Jack_MountingPin, Connector_BarrelJack:BarrelJack_Horizontal, symbol Connector:Barrel_Jack_MountingPin
- C1: footprint pj-bis2025:LDO_5V_out_TAJR105K016RNJAC_TAJR_AVX -> pj-bis2025:tantal_TAJR105K016RNJ_TAJR_AVX-M
Connections:
- net AIN1N_in- is gone; now on net AIN1N_in: C15.2, Re9.2
- net AIN1P_in+ is gone; now on net AIN1P_in: C15.1, Re11.2
- net diff1_in_N: no longer names the net of C13.1, Re12.2, Re13.1, Re14.1
- net diff1_in_P: no longer names the net of C13.2, Re5.1, Re6.2, Re7.1
- net diff1_out_N: no longer names the net of C11.1, Re8.1, U4.15 (VOUT1-)
- net diff1_out_P: no longer names the net of C17.1, Re10.1, U4.14 (VOUT1+)
- net diff2_in_N: no longer names the net of C14.1, C17.2, Re13.2, U4.3 (VIN1-)
- net diff2_in_P: no longer names the net of C11.2, C14.2, Re7.2, U4.2 (VIN1+)
- net diff2_out_N: no longer names the net of Re5.2, Re8.2, Re9.1
- net diff2_out_P: no longer names the net of Re10.2, Re11.1, Re14.2
- net diff3_in_N: no longer names the net of C20.1, Re22.2, Re23.1, Re24.1
- net diff3_in_P: no longer names the net of C20.2, Re15.1, Re16.2, Re17.1
- net diff3_out_N: no longer names the net of C18.1, Re18.1, U4.11 (VOUT2-)
- net diff3_out_P: no longer names the net of C24.1, Re20.1, U4.10 (VOUT2+)
- net diff4_in_N: no longer names the net of C21.1, C24.2, Re23.2, U4.7 (VIN2-)
- net diff4_in_P: no longer names the net of C18.2, C21.2, Re17.2, U4.6 (VIN2+)
- net diff4_out_N: no longer names the net of Re15.2, Re18.2, Re19.1
- net diff4_out_P: no longer names the net of Re20.2, Re21.1, Re24.2
Other:
- company: senserity -> (none)
- title: pj-bis2025 -> (none)
- moved on the sheet: C1, C10, C11, C12, C13, C14, C15, C16, C17, C18, C19, C2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
